File: kicad_project/janus.kicad_pcb (KiCad board)
At the start: 2 copper layers, 180.2 x 117.5 mm, 55 parts

Commit message: generated files
Connections:
- T1 pad 2: RAW -> VCC
Other:
- outline, holes or cut-outs redrawn
Changed lines of the file:
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@@
           (pad "" np_thru_hole circle (at -1.5 0) (size 1 1) (drill 0.9) (layers *.Cu *.Mask))
           (pad 1 smd rect (at 2.25 2.075 -90) (size 0.9 1.25) (layers F.Cu F.Paste F.Mask) (net 48 "BPOS"))
-          (pad 2 smd rect (at -0.75 2.075 -90) (size 0.9 1.25) (layers F.Cu F.Paste F.Mask) (net 37 "RAW"))
+          (pad 2 smd rect (at -0.75 2.075 -90) (size 0.9 1.25) (layers F.Cu F.Paste F.Mask) (net 40 "VCC"))
           (pad 3 smd rect (at -2.25 2.075 -90) (size 0.9 1.25) (layers F.Cu F.Paste F.Mask))
           (pad 1 smd rect (at -2.25 2.075 -90) (size 0.9 1.25) (layers B.Cu B.Paste B.Mask) (net 48 "BPOS"))
-          (pad 2 smd rect (at 0.75 2.075 -90) (size 0.9 1.25) (layers B.Cu B.Paste B.Mask) (net 37 "RAW"))
+          (pad 2 smd rect (at 0.75 2.075 -90) (size 0.9 1.25) (layers B.Cu B.Paste B.Mask) (net 40 "VCC"))
           (pad 3 smd rect (at 2.25 2.075 -90) (size 0.9 1.25) (layers B.Cu B.Paste B.Mask))
           (pad "" smd rect (at 3.7 -1.1 -90) (size 0.9 0.9) (layers F.Cu F.Paste F.Mask))
@@
 (gr_line (start 126.4117054583427 152.7508965304989) (end 43.48745579999999 166.63336469999996) (angle 90) (layer Edge.Cuts) (width 0.15))
 (gr_arc (start 42.4967739 160.7157174) (end 36.5879274 161.75760649999998) (angle -89.50383659124697) (layer Edge.Cuts) (width 0.15))
-(gr_circle (center 27.9674082 84.07436080000001) (end 29.9674082 84.07436080000001) (layer Edge.Cuts) (width 0.15))
-(gr_circle (center 96.5509974 62.562997199999955) (end 98.5509974 62.562997199999955) (layer Edge.Cuts) (width 0.15))
-(gr_circle (center 180.64783640000002 64.77356459999999) (end 182.64783640000002 64.77356459999999) (layer Edge.Cuts) (width 0.15))
-(gr_circle (center 180.64783640000002 127.27356459999999) (end 182.64783640000002 127.27356459999999) (layer Edge.Cuts) (width 0.15))
-(gr_circle (center 125.6975091 147.17006139999998) (end 127.6975091 147.17006139999998) (layer Edge.Cuts) (width 0.15))
-(gr_circle (center 41.6856144 161.8741733) (end 43.6856144 161.8741733) (layer Edge.Cuts) (width 0.15))
 )

Commit message: routed and completed
Parts:
- moved S6 111.6 mm to (171.1, 161.3)
- moved S11 111.6 mm to (187.6, 134.6)
- moved MCU1 111.6 mm to (272.8, 112.9)
- moved S22 111.6 mm to (251.3, 110.9)
- moved D3 111.6 mm to (156.7, 140.0)
- moved S14 111.6 mm to (209.2, 148.2)
- moved D10 111.6 mm to (198.4, 146.7)
- moved D5 111.6 mm to (182.3, 173.1)
- moved B1 111.6 mm to (272.8, 149.9)
- moved D8 111.6 mm to (172.2, 115.4)
- moved S1 111.6 mm to (155.6, 185.9)
- moved D25 111.6 mm to (292.1, 198.9)
- moved S2 111.6 mm to (152.3, 166.7)
- moved S9 111.6 mm to (193.0, 173.2)
- moved S16 111.6 mm to (203.8, 109.6)
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Connections:
- MCU1 pad : P9 -> 14
- OLED1 pad : P1 -> O5
- OLED1 pad 1: (no net) -> O1
- OLED1 pad 2: (no net) -> O2
- OLED1 pad 4: (no net) -> O4
- OLED1 pad 5: (no net) -> O5
- S1 pad 1: P15 -> P20
- S10 pad 1: P16 -> P18
- S11 pad 1: P16 -> P18
- S12 pad 1: P16 -> P18
- S13 pad 1: P10 -> P15
- S14 pad 1: P10 -> P15
- S15 pad 1: P10 -> P15
- S16 pad 1: P10 -> P15
- S17 pad 1: P20 -> P14
- S18 pad 1: P20 -> P14
- S19 pad 1: P20 -> P14
- S2 pad 1: P15 -> P20
- S20 pad 1: P19 -> P16
- S21 pad 1: P19 -> P16
- S22 pad 1: P19 -> P16
- S23 pad 1: P20 -> P14
- S24 pad 1: P19 -> P16
- S25 pad 1: P18 -> P10
- S3 pad 1: P15 -> P20
- S4 pad 1: P15 -> P20
- S5 pad 1: P14 -> P19
- S6 pad 1: P14 -> P19
- S7 pad 1: P14 -> P19
- S8 pad 1: P14 -> P19
- S9 pad 1: P16 -> P18
- T1 pad 2: VCC -> RAW
Routing:
- net P20: track 0.00 -> 294.8 mm
- net P19: track 0.00 -> 274.3 mm
- net P9: track 0.00 -> 261.4 mm
- net P18: track 0.00 -> 253.3 mm
- net P15: track 0.00 -> 233.2 mm
- net P14: track 0.00 -> 221.1 mm
- net P16: track 0.00 -> 200.2 mm
- net P6: track 0.00 -> 175.6 mm
- net P8: track 0.00 -> 169.0 mm
- net P7: track 0.00 -> 157.4 mm
- net GND: track 0.00 -> 118.4 mm, vias 0 -> 1
- net P10: track 0.00 -> 102.9 mm, vias 0 -> 1
- net RST: track 0.00 -> 77.7 mm, vias 0 -> 3
- net RAW: track 0.00 -> 72.8 mm, vias 0 -> 1
- net P1: track 0.00 -> 66.0 mm, vias 0 -> 2
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Other:
- outline, holes or cut-outs redrawn
- net class Default removed
- rule pad_to_mask_clearance: 0.05 -> 0
